File: B0505/B0505.kicad_sch (KiCad schematic)
At the start: 22 parts, among them J1 CN-TB-3.5MM-2P-M-TH-ST, J2 CN-BERG-2.54MM-2P-M-TH-ST, J3 CN-BERG-2.54MM-2P-M-TH-ST, J4 CN-TB-3.5MM-2P-M-TH-ST

Commit message: moved holes and changed gnd near d6
Other:
- moved on the sheet: H1, H2, H3, H4
Changed lines of the file:
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@@
 	(symbol
 		(lib_id "Mechanical:MountingHole")
-		(at 186.309 64.643 0)
+		(at 181.864 76.327 0)
 		(unit 1)
 		(exclude_from_sim no)
@@
 		(dnp no)
 		(property "Reference" "H4"
-			(at 188.849 63.373 0)
+			(at 184.404 75.057 0)
 			(effects
 				(font
@@
 		)
 		(property "Value" "MountingHole"
-			(at 180.594 68.453 0)
+			(at 176.149 80.137 0)
 			(effects
 				(font
@@
 		)
 		(property "Footprint" "MountingHole:MountingHole_3.2mm_M3"
-			(at 186.309 64.643 0)
-			(effects
-				(font
-					(size 1.27 1.27)
-				)
-				(hide yes)
-			)
-		)
-		(property "Datasheet" "~"
-			(at 186.309 64.643 0)
+			(at 181.864 76.327 0)
+			(effects
+				(font
+					(size 1.27 1.27)
+				)
+				(hide yes)
+			)
+		)
+		(property "Datasheet" "~"
+			(at 181.864 76.327 0)
 			(effects
 				(font
@@
 		)
 		(property "Description" ""
-			(at 186.309 64.643 0)
+			(at 181.864 76.327 0)
 			(effects
 				(font
@@
 	(symbol
 		(lib_id "Mechanical:MountingHole")
-		(at 150.749 64.008 0)
+		(at 146.304 75.692 0)
 		(unit 1)
 		(exclude_from_sim no)
@@
 		(dnp no)
 		(property "Reference" "H2"
-			(at 153.289 62.738 0)
+			(at 148.844 74.422 0)
 			(effects
 				(font
@@
 		)
 		(property "Value" "MountingHole"
-			(at 145.034 67.818 0)
+			(at 140.589 79.502 0)
 			(effects
 				(font
@@
 		)
 		(property "Footprint" "MountingHole:MountingHole_3.2mm_M3"
-			(at 150.749 64.008 0)
-			(effects
-				(font
-					(size 1.27 1.27)
-				)
-				(hide yes)
-			)
-		)
-		(property "Datasheet" "~"
-			(at 150.749 64.008 0)
+			(at 146.304 75.692 0)
+			(effects
+				(font
+					(size 1.27 1.27)
+				)
+				(hide yes)
+			)
+		)
+		(property "Datasheet" "~"
+			(at 146.304 75.692 0)
 			(effects
 				(font
@@
 		)
 		(property "Description" ""
-			(at 150.749 64.008 0)
+			(at 146.304 75.692 0)
 			(effects
 				(font
@@
 	(symbol
 		(lib_id "Mechanical:MountingHole")
-		(at 133.604 64.008 0)
+		(at 129.159 75.692 0)
 		(unit 1)
 		(exclude_from_sim no)
@@
 		(dnp no)
 		(property "Reference" "H1"
-			(at 136.144 62.738 0)
+			(at 131.699 74.422 0)
 			(effects
 				(font
@@
 		)
 		(property "Value" "MountingHole"
-			(at 127.889 67.818 0)
+			(at 123.444 79.502 0)
 			(effects
 				(font
@@
 		)
 		(property "Footprint" "MountingHole:MountingHole_3.2mm_M3"
-			(at 133.604 64.008 0)
-			(effects
-				(font
-					(size 1.27 1.27)
-				)
-				(hide yes)
-			)
-		)
-		(property "Datasheet" "~"
-			(at 133.604 64.008 0)
+			(at 129.159 75.692 0)
+			(effects
+				(font
+					(size 1.27 1.27)
+				)
+				(hide yes)
+			)
+		)
+		(property "Datasheet" "~"
+			(at 129.159 75.692 0)
 			(effects
 				(font
@@
 		)
 		(property "Description" ""
-			(at 133.604 64.008 0)
+			(at 129.159 75.692 0)
 			(effects
 				(font
@@
 	(symbol
 		(lib_id "Mechanical:MountingHole")
-		(at 168.529 64.008 0)
+		(at 164.084 75.692 0)
 		(unit 1)
 		(exclude_from_sim no)
@@
 		(dnp no)
 		(property "Reference" "H3"
-			(at 171.069 62.738 0)
+			(at 166.624 74.422 0)
 			(effects
 				(font
@@
 		)
 		(property "Value" "MountingHole"
-			(at 162.814 67.818 0)
+			(at 158.369 79.502 0)
 			(effects
 				(font
@@
 		)
 		(property "Footprint" "MountingHole:MountingHole_3.2mm_M3"
-			(at 168.529 64.008 0)
-			(effects
-				(font
-					(size 1.27 1.27)
-				)
-				(hide yes)
-			)
-		)
-		(property "Datasheet" "~"
-			(at 168.529 64.008 0)
+			(at 164.084 75.692 0)
+			(effects
+				(font
+					(size 1.27 1.27)
+				)
+				(hide yes)
+			)
+		)
+		(property "Datasheet" "~"
+			(at 164.084 75.692 0)
 			(effects
 				(font
@@
 		)
 		(property "Description" ""
-			(at 168.529 64.008 0)
-			(effects
-				(font
+			(at 164.084 75.692 0)
+			(effects
+				(font
